Commit message: Rebuild Time

File: final_description/robots/final_gazebo.urdf (robot description, URDF)
Before this commit: robot final, 5 links, 4 joints
Links:
- added link left_caster_link, mass 0.0814912470443748; collision mesh filename=package://final_description/meshes/left_caster_link.STL; visual mesh filename=package://final_description/meshes/left_caster_link.STL
- added link right_caster_link, mass 0.0814912470443749; collision mesh filename=package://final_description/meshes/right_caster_link.STL; visual mesh filename=package://final_description/meshes/right_caster_link.STL
- link base_link: mass 4.14818186398938 -> 12.6996504557446
- link rear_caster_link: mass 0.176949617511378 -> 0.013967106304125
Joints:
- added joint left_caster_joint: type continuous, parent rear_caster_link, child left_caster_link, origin xyz=0 0 0 rpy=0 0 0, axis 0 -1 0
- added joint right_caster_joint: type continuous, parent rear_caster_link, child right_caster_link, origin xyz=0.014747 -0.035382 -0.010031 rpy=-1.3002 -5.9492E-33 1.5708, axis -1 0 0
- joint laser_joint: origin xyz=-0.0109499999999999 0 0.25575 rpy=1.45390373192998E-33 -3.44227613947609E-17 -4.22366966803326E-17 -> xyz=-0.01095 0 0.25575 rpy=1.4539E-33 -3.4423E-17 -4.2237E-17
- joint left_wheel_joint: origin xyz=0 0.1997875 0 rpy=0 -3.44227613947609E-17 0 -> xyz=0 0.19979 0 rpy=0 -3.4423E-17 0
- joint rear_caster_joint: origin xyz=-0.311952216057906 0 -0.00604000000000001 rpy=-3.04704848392389E-33 -1.0830817995158E-17 8.85184209651363E-17 -> xyz=-0.31195 0 -0.00604 rpy=-3.047E-33 -1.0831E-17 8.8518E-17
- joint right_wheel_joint: origin xyz=0 -0.202910199564064 0 rpy=0 -3.44227613947609E-17 0 -> xyz=0 -0.20291 0 rpy=0 -3.4423E-17 0
